Commit message: update

File: icl_ur5_setup_description/robots/ur5_robotiq_140_joint_limited.xacro (robot description, xacro)
@@ -9,5 +9,5 @@
     <!-- arm -->
     <xacro:ur5_robot prefix="${prefix}" joint_limited="true"
-      shoulder_pan_lower_limit="${-3*pi/4}" shoulder_pan_upper_limit="${pi/2}"
+      shoulder_pan_lower_limit="${-pi}" shoulder_pan_upper_limit="${pi}"
       shoulder_lift_lower_limit="${-pi*7/8}" shoulder_lift_upper_limit="${-pi/8}"
       elbow_joint_lower_limit="${-pi}" elbow_joint_upper_limit="${pi}"

File: icl_ur5_setup_description/urdf/robotiq_arg2f_140_model_macro.xacro (robot description, xacro)
@@ -159,5 +159,5 @@
       <axis xyz="-1 0 0" />
       <!-- <limit lower="-3.14159" upper="3.14159" velocity="2.0" effort="1000" /> -->
-      <limit lower="0" upper="0.775" velocity="2.0" effort="1000" />
+      <limit lower="0" upper="0.85" velocity="2.0" effort="1000" />
     </joint>
     <xacro:finger_joints prefix="${prefix}" fingerprefix="left" reflect="1.0"/>

Commit message: enlarge shoulder_pan joint limit

File: icl_ur5_setup_description/robots/ur5_robotiq_140_joint_limited.xacro (robot description, xacro)
@@ -9,8 +9,8 @@
     <!-- arm -->
     <xacro:ur5_robot prefix="${prefix}" joint_limited="true"
-      shoulder_pan_lower_limit="${-pi}" shoulder_pan_upper_limit="${pi}"
-      shoulder_lift_lower_limit="${-pi*7/8}" shoulder_lift_upper_limit="${-pi/8}"
+      shoulder_pan_lower_limit="${-pi * 3/2 }" shoulder_pan_upper_limit="${pi*3/2}"
+      shoulder_lift_lower_limit="${-pi}" shoulder_lift_upper_limit="${pi}"
       elbow_joint_lower_limit="${-pi}" elbow_joint_upper_limit="${pi}"
-      wrist_1_lower_limit="${-pi}" wrist_1_upper_limit="${pi}"
+      wrist_1_lower_limit="${-pi*3/2}" wrist_1_upper_limit="${pi/2}"
       wrist_2_lower_limit="${-pi}" wrist_2_upper_limit="${pi}"
       wrist_3_lower_limit="${-pi}" wrist_3_upper_limit="${pi}"
@@ -23,5 +23,5 @@
       <parent link= "world" />
       <child link = "${prefix}base_link" />
-      <origin xyz="0.0 0.0 0.0" rpy="0.0 0.0 0.0" />
+      <origin xyz="0.0 0.0 0.0" rpy="0.0 0.0 ${pi/2}" />
     </joint>
     <!--force torque sensor-->

Commit message: fix robot_state_publisher errer

File: icl_ur5_setup_description/robots/ur5_robotiq_140_joint_limited.xacro (robot description, xacro)
@@ -16,9 +16,6 @@
       wrist_3_lower_limit="${-pi}" wrist_3_upper_limit="${pi}"
     />
-    <!-- gripper -->
-    <xacro:robotiq_arg2f_140 prefix="${prefix}" />
-    <!--dummy link-->
-  	<link name="world" />
-    <joint name="fixed_link-robot_base" type="fixed">
+    <link name="world" />
+    <joint name="fixed_link_robot_base" type="fixed">
       <parent link= "world" />
       <child link = "${prefix}base_link" />
@@ -29,5 +26,7 @@
       <origin xyz="0.009 0 0 " rpy="-${pi/2} 0 -${pi/2}"/>
     </xacro:robotiq_fts150>
-    <joint name="ur5_ee_link-gripper_base" type="fixed">
+   <!-- gripper -->
+    <xacro:robotiq_arg2f_140 prefix="${prefix}" />
+    <joint name="ur5_ee_link_gripper_base" type="fixed">
       <parent link= "${prefix}fts_toolside" />
       <child link = "${prefix}robotiq_arg2f_base_link" />
@@ -38,5 +37,5 @@
       <parent link= "${prefix}ee_link" />
       <child link = "${prefix}tool" />
-      <origin xyz=" 0.00 0.0 0.1" rpy="0.0 0.0 0.0" />
+      <origin xyz=" 0.00 0.0 0.2" rpy="0.0 0.0 0.0" />
     </joint>
   </xacro:macro>
